Commit message: initial commit

File: my_robot/urdf/my_robot.xacro (robot description, xacro)
@@ -124,5 +124,5 @@
    </link>
     <joint type="fixed" name="hokuyo_joint">
-    	<origin xyz="0 0 0.15" rpy="0 0 0"/>
+    	<origin xyz="0 0 0.16" rpy="0 0 0"/>
    	  <child link="hokuyo"/>
     	<parent link="chassis"/>

Commit message: Moved screenshots and corrected footprint

File: my_robot/urdf/my_robot.xacro (robot description, xacro)
@@ -10,5 +10,5 @@
   <link name="robot_footprint"></link>
   <joint name="robot_footprint_joint" type="fixed">
-    <origin xyz="0 0 0" rpy="0 0 0" />
+    <origin xyz="0 0 0" rpy="0 0 3.1415" />
     <parent link="robot_footprint"/>
     <child link="chassis" />
